Commit message: pingu & cubo

File: source/isaaclab_assets/data/Robots/SpaceR-TheDreamLab/Pingu/pingu.urdf (robot description, URDF)
Before this commit: robot pingu_v3, 14 links, 14 joints
Links:
- added link thruster_1_link; visual cylinder length=0.055 radius=0.006
- added link thruster_2_link; visual cylinder length=0.055 radius=0.006
- added link thruster_3_link; visual cylinder length=0.055 radius=0.006
- added link thruster_4_link; visual cylinder length=0.055 radius=0.006
- added link thruster_5_link; visual cylinder length=0.055 radius=0.006
- added link thruster_6_link; visual cylinder length=0.055 radius=0.006
- added link thruster_7_link; visual cylinder length=0.055 radius=0.006
- added link thruster_8_link; visual cylinder length=0.055 radius=0.006
- added link world
- link anchor_link: mass 0.0001 -> None; geometry 
- link base_link: geometry collision mesh filename=package://pingu_description/mesh/base_link.stl scale=0.001 0.001 0.001; visual mesh filename=package://pingu_description/mesh/base_link.stl scale=0.001 0.001 0.001
- link rw_base: mass 1.0 -> None; geometry 
- link rw_rotor: geometry visual cylinder length=0.008 radius=0.1
- link x_lock_link: mass 0.0001 -> None; geometry 
- link y_lock_link: mass 0.0001 -> None; geometry 
Joints:
- removed joint rw_joint
- added joint rw_revolute_joint: type revolute, parent rw_base, child rw_rotor, origin xyz=0 0 0.05 rpy=0 0 0, axis 0 0 1, limit lower=-1e9 upper=1e9 effort=10.0 velocity=100
- added joint thruster_1_joint: type fixed, parent base_link, child thruster_1_link, origin xyz=-0.168 0.168 0.295 rpy=1.57079632675 0 -0.785398163375
- added joint thruster_2_joint: type fixed, parent base_link, child thruster_2_link, origin xyz=-0.168 0.168 0.305 rpy=-1.57079632675 0 0.785398163375
- added joint thruster_3_joint: type fixed, parent base_link, child thruster_3_link, origin xyz=0.168 0.168 0.295 rpy=-1.57079632675 0 -0.785398163375
- added joint thruster_4_joint: type fixed, parent base_link, child thruster_4_link, origin xyz=0.168 0.168 0.305 rpy=1.57079632675 0 0.785398163375
- added joint thruster_5_joint: type fixed, parent base_link, child thruster_5_link, origin xyz=0.168 -0.168 0.305 rpy=-1.57079632675 0 0.785398163375
- added joint thruster_6_joint: type fixed, parent base_link, child thruster_6_link, origin xyz=0.168 -0.168 0.295 rpy=1.57079632675 0 -0.785398163375
- added joint thruster_7_joint: type fixed, parent base_link, child thruster_7_link, origin xyz=-0.168 -0.168 0.305 rpy=1.57079632675 0 0.785398163375
- added joint thruster_8_joint: type fixed, parent base_link, child thruster_8_link, origin xyz=-0.168 -0.168 0.295 rpy=-1.57079632675 0 -0.785398163375
- joint anchor_joint: origin xyz=0 0 0.2 rpy=0 0 0 -> xyz=0 0 0.05 rpy=0 0 0; parent robot -> world
- joint base_joint: origin xyz=0 0 0.1 rpy=0 0 0 -> xyz=0 0 0 rpy=0 0 0
- joint left_base_joint: origin xyz=0.18384776309900003 0.18384776309900003 .3475 rpy=0 0 0.785398163375 -> xyz=0.26 0 .3475 rpy=0 0 0
- joint right_base_joint: origin xyz=0.18384776309900003 -0.18384776309900003 .3475 rpy=0 0 -0.785398163375 -> xyz=0 -0.26 .3475 rpy=0 0 -1.57079632675
